File: Hardware/APRN_Relay/APRNModem.kicad_sch (KiCad schematic)
At the start: 7 parts

Commit message: Cleanup DRA footprint
Parts:
- gave numbers to parts that had none: 7
Changed lines of the file:
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@@
   (symbol (lib_id "Device:R_Small") (at 255.27 158.115 90) (unit 1)
     (in_bom yes) (on_board yes)
-    (property "Reference" "R?" (id 0) (at 255.27 160.655 90))
+    (property "Reference" "R201" (id 0) (at 255.27 160.655 90))
     (property "Value" "2K2" (id 1) (at 255.27 155.575 90))
     (property "Footprint" "Resistor_SMD:R_0805_2012Metric" (id 2) (at 255.27 158.115 0)
@@
   (symbol (lib_id "Device:C_Small") (at 185.42 70.485 0) (unit 1)
     (in_bom yes) (on_board yes) (fields_autoplaced)
-    (property "Reference" "C?" (id 0) (at 187.96 69.2212 0)
+    (property "Reference" "C201" (id 0) (at 187.96 69.2212 0)
       (effects (font (size 1.27 1.27)) (justify left))
     )
@@
   (symbol (lib_id "KenwoodFox:DRA818V") (at 202.565 99.06 0) (unit 1)
     (in_bom yes) (on_board yes)
-    (property "Reference" "U?" (id 0) (at 208.915 122.555 0))
+    (property "Reference" "U201" (id 0) (at 208.915 122.555 0))
     (property "Value" "DRA818V" (id 1) (at 208.28 78.74 0))
     (property "Footprint" "KenwoodFox:DRA818V" (id 2) (at 203.835 123.19 0)
@@
   (symbol (lib_id "power:GND") (at 266.7 92.71 0) (unit 1)
     (in_bom yes) (on_board yes)
-    (property "Reference" "#PWR?" (id 0) (at 266.7 99.06 0)
+    (property "Reference" "#PWR0209" (id 0) (at 266.7 99.06 0)
       (effects (font (size 1.27 1.27)) hide)
     )
@@
   (symbol (lib_id "Device:C_Small") (at 194.31 70.485 0) (unit 1)
     (in_bom yes) (on_board yes) (fields_autoplaced)
-    (property "Reference" "C?" (id 0) (at 196.85 69.2212 0)
+    (property "Reference" "C202" (id 0) (at 196.85 69.2212 0)
       (effects (font (size 1.27 1.27)) (justify left))
     )
@@
   (symbol (lib_id "power:+3.3V") (at 251.46 156.845 0) (unit 1)
     (in_bom yes) (on_board yes)
-    (property "Reference" "#PWR?" (id 0) (at 251.46 160.655 0)
+    (property "Reference" "#PWR0208" (id 0) (at 251.46 160.655 0)
       (effects (font (size 1.27 1.27)) hide)
     )
@@
   (symbol (lib_id "power:GND") (at 194.31 74.295 0) (unit 1)
     (in_bom yes) (on_board yes)
-    (property "Reference" "#PWR?" (id 0) (at 194.31 80.645 0)
+    (property "Reference" "#PWR0204" (id 0) (at 194.31 80.645 0)
       (effects (font (size 1.27 1.27)) hide)
     )
@@
   (symbol (lib_id "power:+4V") (at 194.31 66.675 0) (unit 1)
     (in_bom yes) (on_board yes)
-    (property "Reference" "#PWR?" (id 0) (at 194.31 70.485 0)
+    (property "Reference" "#PWR0203" (id 0) (at 194.31 70.485 0)
       (effects (font (size 1.27 1.27)) hide)
     )
@@
   (symbol (lib_id "Connector:Conn_Coaxial") (at 266.7 82.55 0) (unit 1)
     (in_bom yes) (on_board yes) (fields_autoplaced)
-    (property "Reference" "J?" (id 0) (at 269.24 81.5731 0)
+    (property "Reference" "J201" (id 0) (at 269.24 81.5731 0)
       (effects (font (size 1.27 1.27)) (justify left))
     )
@@
   (symbol (lib_id "power:+4V") (at 202.565 66.675 0) (unit 1)
     (in_bom yes) (on_board yes)
-    (property "Reference" "#PWR?" (id 0) (at 202.565 70.485 0)
+    (property "Reference" "#PWR0205" (id 0) (at 202.565 70.485 0)
       (effects (font (size 1.27 1.27)) hide)
     )
@@
   (symbol (lib_id "power:GND") (at 246.38 97.79 0) (unit 1)
     (in_bom yes) (on_board yes)
-    (property "Reference" "#PWR?" (id 0) (at 246.38 104.14 0)
+    (property "Reference" "#PWR0207" (id 0) (at 246.38 104.14 0)
       (effects (font (size 1.27 1.27)) hide)
     )
@@
   (symbol (lib_id "Device:LED") (at 262.89 158.115 180) (unit 1)
     (in_bom yes) (on_board yes)
-    (property "Reference" "D?" (id 0) (at 262.89 160.655 0))
+    (property "Reference" "D201" (id 0) (at 262.89 160.655 0))
     (property "Value" "RX" (id 1) (at 262.89 155.575 0))
     (property "Footprint" "LED_SMD:LED_0805_2012Metric" (id 2) (at 262.89 158.115 0)
@@
   (symbol (lib_id "power:+4V") (at 185.42 66.675 0) (unit 1)
     (in_bom yes) (on_board yes)
-    (property "Reference" "#PWR?" (id 0) (at 185.42 70.485 0)
+    (property "Reference" "#PWR0201" (id 0) (at 185.42 70.485 0)
       (effects (font (size 1.27 1.27)) hide)
     )
@@
   (symbol (lib_id "power:GND") (at 203.2 124.46 0) (unit 1)
     (in_bom yes) (on_board yes) (fields_autoplaced)
-    (property "Reference" "#PWR?" (id 0) (at 203.2 130.81 0)
+    (property "Reference" "#PWR0206" (id 0) (at 203.2 130.81 0)
       (effects (font (size 1.27 1.27)) hide)
     )
@@
   (symbol (lib_id "power:GND") (at 185.42 74.295 0) (unit 1)
     (in_bom yes) (on_board yes)
-    (property "Reference" "#PWR?" (id 0) (at 185.42 80.645 0)
+    (property "Reference" "#PWR0202" (id 0) (at 185.42 80.645 0)
       (effects (font (size 1.27 1.27)) hide)
     )
@@
   (symbol (lib_id "RF_Filter:LFCN-490") (at 246.38 82.55 0) (unit 1)
     (in_bom yes) (on_board yes)
-    (property "Reference" "FL?" (id 0) (at 252.73 91.44 0))
+    (property "Reference" "FL201" (id 0) (at 252.73 91.44 0))
     (property "Value" "LFCN-490" (id 1) (at 243.84 73.66 0))
     (property "Footprint" "Filter:Filter_Mini-Circuits_FV1206" (id 2) (at 246.38 69.85 0)

Commit message: Even prettier
Parts:
- removed C201: 4.7u, Capacitor_SMD:C_0805_2012Metric, symbol Device:C_Small
- removed C202: 100p, Capacitor_SMD:C_0805_2012Metric, symbol Device:C_Small
- added C?: 100p, Capacitor_SMD:C_0805_2012Metric, symbol Device:C_Small
- added C?: 4.7u, Capacitor_SMD:C_0805_2012Metric, symbol Device:C_Small
Connections:
- net +4V: now also C?.2, C?.2
- net GND: now also C?.1, C?.1
- net RXD renamed DRA_RX
- net TXD renamed DRA_TX
Other:
- note added: "Not 3.3v or 5v!"
- note removed: "Not 3.3v!"
- moved on the sheet: FL201, J201, U201

Commit message: Do hardware things
Parts:
- added C201: 1uF, Capacitor_SMD:C_0805_2012Metric, symbol Device:C_Small
- added R201, R? (x2): 100K, Resistor_SMD:R_0805_2012Metric, symbol Device:R_Small
- added U201: VS1003, Package_QFP:LQFP-48_7x7mm_P0.5mm, symbol KenwoodFox:VS1003
- C202: renamed from C?; value 100p -> 100pF
- C203: renamed from C?; value 4.7u -> 4.7uF
- renumbered R201 to R202, U201 to U202
Connections:
- net GND: now also C201.1, R201.2, R?.2, U201.16 (DGND1), U201.20 (DGND2), U201.21 (DGND3), U201.22 (DGND4), U201.37 (AGND0), U201.4 (DGND0), U201.40 (AGND1), U201.41 (AGND2), U201.47 (AGND3)
- new net: C201.2, U201.44 (RCAP)
- new net: R201.1, U201.33 (GPIO0)
- new net: R?.2, U201.26 (RXD)
- new net AVDD: U201.38 (AVDD0), U201.43 (AVDD1), U201.45 (AVDD2)
- new net CVDD: U201.24 (CVDD2), U201.31 (CVDD3), U201.5 (CVDD0), U201.7 (CVDD1)
- new net DREQ: U201.8 (DREQ)
- new net IOVDD: R?.1, U201.14 (IOVDD1), U201.19 (IOVDD2), U201.32 (TEST), U201.6 (IOVDD0)
- new net SCLK: U201.28 (SCLK)
- new net SI: U201.29 (SI)
- new net SO: U201.30 (SO)
- new net ~{xCS}: U201.23 (~{xCS})
- new net ~{xDCS}: U201.13 (~{xDCS})
- new net ~{xRESET}: R?.1, U201.3 (~{xRESET})
- no-connect marks 0 -> 5
Other:
- note added: "Audio"
- note added: "Indicators"
- note added: "Radio"
- moved on the sheet: C202, C203, FL201, J201, U202
