File: Hardware/APRN_Relay/APRN_Relay.kicad_pcb (KiCad board)
At the start: 2 copper layers, 7 parts, among them J201 Conn_Coaxial, U201 DRA818V

Commit message: Do hardware things
Parts:
- added C201: 1uF, Capacitor_SMD:C_0805_2012Metric, F.Cu at (170.4, 96.3)
- added C202: 100pF, Capacitor_SMD:C_0805_2012Metric, F.Cu at (170.4, 99.3)
- added C203: 4.7uF, Capacitor_SMD:C_0805_2012Metric, F.Cu at (174.9, 96.3)
- added R201: 100K, Resistor_SMD:R_0805_2012Metric, F.Cu at (170.4, 102.3)
- added U201: VS1003, Package_QFP:LQFP-48_7x7mm_P0.5mm, F.Cu at (162.5, 100.4)
- renumbered R201 to R202, U201 to U202
Connections:
- net /APRN Modem/RXD renamed /APRN Modem/DRA_RX
- net /APRN Modem/TXD renamed /APRN Modem/DRA_TX
