File: Hardware/APRN_Relay/APRN_Relay.kicad_sch (KiCad schematic)
At the start: 0 parts

Commit message: Add some things for the vs1003
Other:
- sheet APRN Modem renamed Modem
- sheet Modem: file APRNModem.kicad_sch -> Modem.kicad_sch
Changed lines of the file:
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@@
 (kicad_sch (version 20211123) (generator eeschema)
   (paper "A4")
-  (sheet (at 121.285 70.485) (size 28.575 46.355) (fields_autoplaced)
+  (sheet (at 121.285 70.485) (size 33.655 24.13) (fields_autoplaced)
     (stroke (width 0.1524) (type solid) (color 0 0 0 0))
     (fill (color 0 0 0 0.0000))
-    (property "Sheet name" "APRN Modem" (id 0) (at 121.285 69.7734 0)
+    (property "Sheet name" "Modem" (id 0) (at 121.285 69.7734 0)
       (effects (font (size 1.27 1.27)) (justify left bottom))
     )
-    (property "Sheet file" "APRNModem.kicad_sch" (id 1) (at 121.285 117.4246 0)
+    (property "Sheet file" "Modem.kicad_sch" (id 1) (at 121.285 95.1996 0)
       (effects (font (size 1.27 1.27)) (justify left top))
     )
@@
     (path "/" (page "1"))
     (path "/e4a26974-393b-4a41-b021-56885f23f4ce" (page "2"))
+    (path "/e4a26974-393b-4a41-b021-56885f23f4ce/b3e8c470-c55e-46e8-9579-d406ff6be8fa" (page "3"))
   )
   (symbol_instances
-    (path "/e4a26974-393b-4a41-b021-56885f23f4ce/c2a4eb15-cc1f-40ff-a34e-8aa78a70bf7f"
-      (reference "#PWR0101") (unit 1) (value "GND") (footprint "")
-    )
-    (path "/e4a26974-393b-4a41-b021-56885f23f4ce/757f4500-5349-4b71-96c8-10e78bbebbce"
-      (reference "#PWR0201") (unit 1) (value "GND") (footprint "")
-    )
-    (path "/e4a26974-393b-4a41-b021-56885f23f4ce/7027166c-897c-4bf9-acbb-9dff2d2232db"
-      (reference "#PWR0202") (unit 1) (value "GND") (footprint "")
-    )
     (path "/e4a26974-393b-4a41-b021-56885f23f4ce/9621d6e5-cfb7-4954-bcd7-ffb29212ebd8"
       (reference "#PWR0203") (unit 1) (value "GND") (footprint "")
@@
       (reference "#PWR0208") (unit 1) (value "GND") (footprint "")
     )
-    (path "/e4a26974-393b-4a41-b021-56885f23f4ce/1752c983-5898-4df5-8736-767ab0df11b2"
+    (path "/e4a26974-393b-4a41-b021-56885f23f4ce/b3e8c470-c55e-46e8-9579-d406ff6be8fa/0146949b-d78a-408b-8319-096b9442ca95"
       (reference "#PWR?") (unit 1) (value "GND") (footprint "")
     )
-    (path "/e4a26974-393b-4a41-b021-56885f23f4ce/1df7cbb2-6c04-423c-ba04-5cff45244c3b"
-      (reference "C201") (unit 1) (value "1uF") (footprint "Capacitor_SMD:C_0805_2012Metric")
+    (path "/e4a26974-393b-4a41-b021-56885f23f4ce/b3e8c470-c55e-46e8-9579-d406ff6be8fa/2397ff79-fe07-4464-a64e-e669110e0eab"
+      (reference "#PWR?") (unit 1) (value "GND") (footprint "")
+    )
+    (path "/e4a26974-393b-4a41-b021-56885f23f4ce/b3e8c470-c55e-46e8-9579-d406ff6be8fa/e2387c31-2146-4d7a-929f-a4439fe4a217"
+      (reference "#PWR?") (unit 1) (value "GND") (footprint "")
+    )
+    (path "/e4a26974-393b-4a41-b021-56885f23f4ce/b3e8c470-c55e-46e8-9579-d406ff6be8fa/e5d23397-9774-407e-b342-36477d8491bb"
+      (reference "#PWR?") (unit 1) (value "GNDA") (footprint "")
+    )
+    (path "/e4a26974-393b-4a41-b021-56885f23f4ce/b3e8c470-c55e-46e8-9579-d406ff6be8fa/fdeab3e9-fe85-4a10-9a45-0e906f24dbd7"
+      (reference "#PWR?") (unit 1) (value "GND") (footprint "")
     )
     (path "/e4a26974-393b-4a41-b021-56885f23f4ce/86372169-1724-4a03-80ab-e5da1b5a62c2"
@@
     (path "/e4a26974-393b-4a41-b021-56885f23f4ce/bf54bad0-10a0-4d3b-be00-02a7b14e2ef8"
       (reference "C203") (unit 1) (value "4.7uF") (footprint "Capacitor_SMD:C_0805_2012Metric")
+    )
+    (path "/e4a26974-393b-4a41-b021-56885f23f4ce/b3e8c470-c55e-46e8-9579-d406ff6be8fa/bcb791db-f472-4d46-b803-d46d3f6d797a"
+      (reference "C?") (unit 1) (value "1uF") (footprint "Capacitor_SMD:C_0805_2012Metric")
+    )
+    (path "/e4a26974-393b-4a41-b021-56885f23f4ce/b3e8c470-c55e-46e8-9579-d406ff6be8fa/bf441614-b9e0-4264-a697-a581bc9aafff"
+      (reference "C?") (unit 1) (value "10uf") (footprint "Capacitor_SMD:CP_Elec_4x3")
     )
     (path "/e4a26974-393b-4a41-b021-56885f23f4ce/c33dbf77-de8f-4986-a43f-ca29c1159491"
@@
       (reference "J201") (unit 1) (value "Conn_Coaxial") (footprint "Connector_Coaxial:SMA_Amphenol_132291_Vertical")
     )
-    (path "/e4a26974-393b-4a41-b021-56885f23f4ce/af309e5b-4862-4302-9b33-42bd4fd6c715"
-      (reference "R201") (unit 1) (value "100K") (footprint "Resistor_SMD:R_0805_2012Metric")
-    )
     (path "/e4a26974-393b-4a41-b021-56885f23f4ce/12606799-4969-48fe-8fbc-0756f39260a6"
       (reference "R202") (unit 1) (value "2K2") (footprint "Resistor_SMD:R_0805_2012Metric")
     )
-    (path "/e4a26974-393b-4a41-b021-56885f23f4ce/c924cc44-c9c0-4f20-ba4d-92621e148eb9"
+    (path "/e4a26974-393b-4a41-b021-56885f23f4ce/b3e8c470-c55e-46e8-9579-d406ff6be8fa/64ead2bd-0817-4de6-8d87-436ab272a9f8"
       (reference "R?") (unit 1) (value "100K") (footprint "Resistor_SMD:R_0805_2012Metric")
     )
-    (path "/e4a26974-393b-4a41-b021-56885f23f4ce/f64a19db-c347-4487-a223-9986dc2d0993"
+    (path "/e4a26974-393b-4a41-b021-56885f23f4ce/b3e8c470-c55e-46e8-9579-d406ff6be8fa/96a4a102-d248-4c40-999c-c18111c2b898"
       (reference "R?") (unit 1) (value "100K") (footprint "Resistor_SMD:R_0805_2012Metric")
     )
-    (path "/e4a26974-393b-4a41-b021-56885f23f4ce/f336105a-4df8-4170-9963-a1bfb83efb91"
-      (reference "U201") (unit 1) (value "VS1003") (footprint "Package_QFP:LQFP-48_7x7mm_P0.5mm")
+    (path "/e4a26974-393b-4a41-b021-56885f23f4ce/b3e8c470-c55e-46e8-9579-d406ff6be8fa/a31b6071-a862-410f-ab96-a4ffb7578e0b"
+      (reference "R?") (unit 1) (value "100K") (footprint "Resistor_SMD:R_0805_2012Metric")
     )
     (path "/e4a26974-393b-4a41-b021-56885f23f4ce/6573725e-f9e6-4a24-91ae-d5a8b834ca14"
       (reference "U202") (unit 1) (value "DRA818V") (footprint "KenwoodFox:DRA818V")
     )
+    (path "/e4a26974-393b-4a41-b021-56885f23f4ce/b3e8c470-c55e-46e8-9579-d406ff6be8fa/08fa121f-1fa0-45b3-b286-1cc666675103"
+      (reference "U?") (unit 1) (value "VS1003") (footprint "Package_QFP:LQFP-48_7x7mm_P0.5mm")
+    )
   )
