File: Hardware/APRN_Relay/Modem.kicad_sch (KiCad schematic)
At the start: 12 parts, among them J201 Conn_Coaxial, U201 VS1003, U202 DRA818V

Commit message: Add some things for the vs1003
Parts:
- removed C201: 1uF, Capacitor_SMD:C_0805_2012Metric, symbol Device:C_Small
- removed R201, R? (x2): 100K, Resistor_SMD:R_0805_2012Metric, symbol Device:R_Small
- removed U201: VS1003, Package_QFP:LQFP-48_7x7mm_P0.5mm, symbol KenwoodFox:VS1003
- C202: value 100pF -> (none); footprint Capacitor_SMD:C_0805_2012Metric -> (none)
- C203: value 4.7uF -> (none); footprint Capacitor_SMD:C_0805_2012Metric -> (none)
- D201: value RX -> (none); footprint LED_SMD:LED_0805_2012Metric -> (none)
- FL201: value LFCN-490 -> (none); footprint Filter:Filter_Mini-Circuits_FV1206 -> (none)
- J201: value Conn_Coaxial -> (none); footprint Connector_Coaxial:SMA_Amphenol_132291_Vertical -> (none)
- R202: value 2K2 -> (none); footprint Resistor_SMD:R_0805_2012Metric -> (none)
- U202: value DRA818V -> (none); footprint KenwoodFox:DRA818V -> (none)
Connections:
- no-connect marks 5 -> 0
Other:
- added sheet VS1003 (VS1003.kicad_sch)
- note removed: "Audio"
- note removed: "Indicators"
- note removed: "Radio"
