File: Hardware/APRN_Modem/DRA818.kicad_sch (KiCad schematic)
At the start: 7 parts

Commit message: Move everything
Parts:
- removed C202, C203: (no value), symbol Device:C_Small
- removed D201: (no value), symbol Device:LED
- removed FL201: (no value), symbol RF_Filter:LFCN-490
- removed J201: (no value), symbol Connector:Conn_Coaxial
- removed R202: (no value), symbol Device:R_Small
- removed U202: (no value), symbol KenwoodFox:DRA818V
- added C?: 100pF, Capacitor_SMD:C_0805_2012Metric, symbol Device:C_Small
- added C?: 4.7uF, Capacitor_SMD:C_0805_2012Metric, symbol Device:C_Small
- added D?: RX, LED_SMD:LED_0805_2012Metric, symbol Device:LED
- added FL?: LFCN-490, Filter:Filter_Mini-Circuits_FV1206, symbol RF_Filter:LFCN-490
- added J?: Conn_Coaxial, Connector_Coaxial:SMA_Amphenol_132291_Vertical, symbol Connector:Conn_Coaxial
- added R?: 2K2, Resistor_SMD:R_0805_2012Metric, symbol Device:R_Small
- added U?: DRA818V, KenwoodFox:DRA818V, symbol KenwoodFox:DRA818V
Connections:
- net +3.3V: now also R?.1
- net +4V: now also C?.2, C?.2, U?.8 (VBAT)
- net DRA_RX: now also U?.16 (RXD)
- net DRA_TX: now also U?.17 (TXD)
- net GND: now also C?.1, C?.1, FL?.2 (GND), FL?.4 (GND), J?.2 (Ext), U?.10 (GND), U?.9 (GND)
- net POWER_TX: now also U?.7 (H/L)
- net PTT: now also U?.5 (PTT)
- net PWR_SAVE: now also U?.6 (PD)
- net RADIO_IN: now also U?.18 (MIC)
- net RADIO_OUT: now also U?.3 (AF_OUT)
- net SQ: now also D?.1 (K), U?.1 (SQ)
- new net: D?.2 (A), R?.2
- new net: FL?.3 (OUT), J?.1 (In)
- new net: FL?.1 (IN), U?.12 (ANT)
Other:
- removed sheet VS1003
- company: (none) -> Kitsune Scientific
- title: (none) -> APRN Modem

Commit message: Clean the rest
Parts:
- gave numbers to parts that had none: 7
Changed lines of the file:
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@@
   (symbol (lib_id "Device:C_Small") (at 193.04 27.305 90) (unit 1)
     (in_bom yes) (on_board yes)
-    (property "Reference" "C?" (id 0) (at 193.04 24.13 90))
+    (property "Reference" "C301" (id 0) (at 193.04 24.13 90))
     (property "Value" "100pF" (id 1) (at 193.04 30.48 90))
     (property "Footprint" "Capacitor_SMD:C_0805_2012Metric" (id 2) (at 193.04 27.305 0)
@@
   (symbol (lib_id "power:GND") (at 200.025 78.74 0) (unit 1)
     (in_bom yes) (on_board yes) (fields_autoplaced)
-    (property "Reference" "#PWR?" (id 0) (at 200.025 85.09 0)
+    (property "Reference" "#PWR0303" (id 0) (at 200.025 85.09 0)
       (effects (font (size 1.27 1.27)) hide)
     )
@@
   (symbol (lib_id "power:GND") (at 186.69 38.1 0) (unit 1)
     (in_bom yes) (on_board yes)
-    (property "Reference" "#PWR?" (id 0) (at 186.69 44.45 0)
+    (property "Reference" "#PWR0301" (id 0) (at 186.69 44.45 0)
       (effects (font (size 1.27 1.27)) hide)
     )
@@
   (symbol (lib_id "Device:R_Small") (at 252.095 157.48 90) (unit 1)
     (in_bom yes) (on_board yes)
-    (property "Reference" "R?" (id 0) (at 252.095 160.02 90))
+    (property "Reference" "R301" (id 0) (at 252.095 160.02 90))
     (property "Value" "2K2" (id 1) (at 252.095 154.94 90))
     (property "Footprint" "Resistor_SMD:R_0805_2012Metric" (id 2) (at 252.095 157.48 0)
@@
   (symbol (lib_id "power:GND") (at 263.525 59.69 0) (unit 1)
     (in_bom yes) (on_board yes)
-    (property "Reference" "#PWR?" (id 0) (at 263.525 66.04 0)
+    (property "Reference" "#PWR0306" (id 0) (at 263.525 66.04 0)
       (effects (font (size 1.27 1.27)) hide)
     )
@@
   (symbol (lib_id "power:+4V") (at 199.39 24.765 0) (unit 1)
     (in_bom yes) (on_board yes)
-    (property "Reference" "#PWR?" (id 0) (at 199.39 28.575 0)
+    (property "Reference" "#PWR0302" (id 0) (at 199.39 28.575 0)
       (effects (font (size 1.27 1.27)) hide)
     )
@@
   (symbol (lib_id "Device:C_Small") (at 193.04 36.195 90) (unit 1)
     (in_bom yes) (on_board yes)
-    (property "Reference" "C?" (id 0) (at 193.04 33.02 90))
+    (property "Reference" "C302" (id 0) (at 193.04 33.02 90))
     (property "Value" "4.7uF" (id 1) (at 193.04 39.37 90))
     (property "Footprint" "Capacitor_SMD:C_0805_2012Metric" (id 2) (at 193.04 36.195 0)
@@
   (symbol (lib_id "Connector:Conn_Coaxial") (at 263.525 49.53 0) (unit 1)
     (in_bom yes) (on_board yes) (fields_autoplaced)
-    (property "Reference" "J?" (id 0) (at 266.065 48.5531 0)
+    (property "Reference" "J301" (id 0) (at 266.065 48.5531 0)
       (effects (font (size 1.27 1.27)) (justify left))
     )
@@
   (symbol (lib_id "KenwoodFox:DRA818V") (at 199.39 60.96 0) (unit 1)
     (in_bom yes) (on_board yes)
-    (property "Reference" "U?" (id 0) (at 204.47 45.72 0))
+    (property "Reference" "U301" (id 0) (at 204.47 45.72 0))
     (property "Value" "DRA818V" (id 1) (at 207.01 76.2 0))
     (property "Footprint" "KenwoodFox:DRA818V" (id 2) (at 200.66 85.09 0)
@@
   (symbol (lib_id "Device:LED") (at 259.715 157.48 180) (unit 1)
     (in_bom yes) (on_board yes)
-    (property "Reference" "D?" (id 0) (at 259.715 160.02 0))
+    (property "Reference" "D301" (id 0) (at 259.715 160.02 0))
     (property "Value" "RX" (id 1) (at 259.715 154.94 0))
     (property "Footprint" "LED_SMD:LED_0805_2012Metric" (id 2) (at 259.715 157.48 0)
@@
   (symbol (lib_id "power:GND") (at 237.49 64.77 0) (unit 1)
     (in_bom yes) (on_board yes)
-    (property "Reference" "#PWR?" (id 0) (at 237.49 71.12 0)
+    (property "Reference" "#PWR0304" (id 0) (at 237.49 71.12 0)
       (effects (font (size 1.27 1.27)) hide)
     )
@@
   (symbol (lib_id "power:+3.3V") (at 248.285 156.21 0) (unit 1)
     (in_bom yes) (on_board yes)
-    (property "Reference" "#PWR?" (id 0) (at 248.285 160.02 0)
+    (property "Reference" "#PWR0305" (id 0) (at 248.285 160.02 0)
       (effects (font (size 1.27 1.27)) hide)
     )
@@
   (symbol (lib_id "RF_Filter:LFCN-490") (at 237.49 49.53 0) (unit 1)
     (in_bom yes) (on_board yes)
-    (property "Reference" "FL?" (id 0) (at 243.84 58.42 0))
+    (property "Reference" "FL301" (id 0) (at 243.84 58.42 0))
     (property "Value" "LFCN-490" (id 1) (at 234.95 40.64 0))
     (property "Footprint" "Filter:Filter_Mini-Circuits_FV1206" (id 2) (at 237.49 36.83 0)
