File: Hardware/APRN_Modem/DRA818.kicad_sch (KiCad schematic)
At the start: 7 parts, among them J301 Conn_Coaxial, U301 DRA818V

Commit message: Bump libs and stuff
Parts:
- J301: footprint Connector_Coaxial:SMA_Amphenol_132291_Vertical -> Connector_Coaxial:SMA_Amphenol_132289_EdgeMount
Changed lines of the file:
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@@
       (effects (font (size 1.27 1.27)) (justify left))
     )
-    (property "Footprint" "Connector_Coaxial:SMA_Amphenol_132291_Vertical" (id 2) (at 263.525 49.53 0)
+    (property "Footprint" "Connector_Coaxial:SMA_Amphenol_132289_EdgeMount" (id 2) (at 263.525 49.53 0)
       (effects (font (size 1.27 1.27)) hide)
     )
