File: Hardware/APRN_Modem/VS1003.kicad_sch (KiCad schematic)
At the start: 6 parts

Commit message: Move everything
Other:
- company: (none) -> Kitsune Scientific
- title: (none) -> APRN Modem
Changed lines of the file:
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@@
 (kicad_sch (version 20211123) (generator eeschema)
   (paper "A4")
+  (title_block
+    (title "APRN Modem")
+    (date "2022-08-01")
+    (rev "${REVISION}")
+    (company "Kitsune Scientific")
+    (comment 4 "Release: ${FULL_REVISION}")
+  )
   (junction (at 146.685 132.715) (diameter 0) (color 0 0 0 0)
   )

Commit message: Clean the rest
Parts:
- gave numbers to parts that had none: 6
Changed lines of the file:
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@@
   (symbol (lib_id "power:GND") (at 168.91 135.255 0) (unit 1)
     (in_bom yes) (on_board yes)
-    (property "Reference" "#PWR?" (id 0) (at 168.91 141.605 0)
+    (property "Reference" "#PWR0204" (id 0) (at 168.91 141.605 0)
       (effects (font (size 1.27 1.27)) hide)
     )
@@
   (symbol (lib_id "KenwoodFox:VS1003") (at 144.145 93.345 0) (unit 1)
     (in_bom yes) (on_board yes)
-    (property "Reference" "U?" (id 0) (at 158.115 59.055 0)
+    (property "Reference" "U201" (id 0) (at 158.115 59.055 0)
       (effects (font (size 1.27 1.27)) (justify left))
     )
@@
   (symbol (lib_id "power:GND") (at 144.145 135.255 0) (unit 1)
     (in_bom yes) (on_board yes)
-    (property "Reference" "#PWR?" (id 0) (at 144.145 141.605 0)
+    (property "Reference" "#PWR0203" (id 0) (at 144.145 141.605 0)
       (effects (font (size 1.27 1.27)) hide)
     )
@@
   (symbol (lib_id "Device:R_Small") (at 121.285 64.77 0) (unit 1)
     (in_bom yes) (on_board yes)
-    (property "Reference" "R?" (id 0) (at 114.3 63.5 0)
+    (property "Reference" "R203" (id 0) (at 114.3 63.5 0)
       (effects (font (size 1.27 1.27)) (justify left))
     )
@@
   (symbol (lib_id "Device:R_Small") (at 111.76 114.3 0) (unit 1)
     (in_bom yes) (on_board yes)
-    (property "Reference" "R?" (id 0) (at 104.775 113.03 0)
+    (property "Reference" "R201" (id 0) (at 104.775 113.03 0)
       (effects (font (size 1.27 1.27)) (justify left))
     )
@@
   (symbol (lib_id "Device:R_Small") (at 120.65 114.3 0) (unit 1)
     (in_bom yes) (on_board yes)
-    (property "Reference" "R?" (id 0) (at 113.665 113.03 0)
+    (property "Reference" "R202" (id 0) (at 113.665 113.03 0)
       (effects (font (size 1.27 1.27)) (justify left))
     )
@@
   (symbol (lib_id "Device:C_Small") (at 168.91 125.095 180) (unit 1)
     (in_bom yes) (on_board yes)
-    (property "Reference" "C?" (id 0) (at 172.085 123.19 0))
+    (property "Reference" "C201" (id 0) (at 172.085 123.19 0))
     (property "Value" "1uF" (id 1) (at 172.085 127 0))
     (property "Footprint" "Capacitor_SMD:C_0805_2012Metric" (id 2) (at 168.91 125.095 0)
@@
   (symbol (lib_id "Device:C_Polarized_Small") (at 184.15 53.975 0) (unit 1)
     (in_bom yes) (on_board yes)
-    (property "Reference" "C?" (id 0) (at 177.165 52.705 0)
+    (property "Reference" "C202" (id 0) (at 177.165 52.705 0)
       (effects (font (size 1.27 1.27)) (justify left))
     )
@@
   (symbol (lib_id "power:GND") (at 111.76 135.255 0) (unit 1)
     (in_bom yes) (on_board yes)
-    (property "Reference" "#PWR?" (id 0) (at 111.76 141.605 0)
+    (property "Reference" "#PWR0201" (id 0) (at 111.76 141.605 0)
       (effects (font (size 1.27 1.27)) hide)
     )
@@
   (symbol (lib_id "power:GNDA") (at 200.66 60.325 0) (unit 1)
     (in_bom yes) (on_board yes) (fields_autoplaced)
-    (property "Reference" "#PWR?" (id 0) (at 200.66 66.675 0)
+    (property "Reference" "#PWR0205" (id 0) (at 200.66 66.675 0)
       (effects (font (size 1.27 1.27)) hide)
     )
@@
   (symbol (lib_id "power:GND") (at 120.65 135.255 0) (unit 1)
     (in_bom yes) (on_board yes)
-    (property "Reference" "#PWR?" (id 0) (at 120.65 141.605 0)
-      (effects (font (size 1.27 1.27)) hide)
-    )
+    (property "Reference" "#PWR0202" (id 0) (at 120.65 141.605 0)
+      (effects (font (size 1.27 1.27)) hide)
+    )
